Commit message: Added extra arm model

File: ragnar_support/urdf/ragnar_upper3_macro.xacro (robot description, xacro)
@@ -51,5 +51,5 @@
   <link name="${prefix}lower_arm_${num}a">
     <visual>
-      <origin xyz="0 0 0" rpy="0 -1.57 3.14" />
+      <origin xyz="0 0 0" rpy="0 0 1.57" />
       <geometry>
         <mesh filename="package://ragnar_support/meshes/ragnar_single_arm2.stl" />
@@ -76,10 +76,19 @@
   <link name="${prefix}lower_arm_${num}b">
     <visual>
-      <origin xyz="0 0 0" rpy="0 0 0" />
+      <origin xyz="0 0 0" rpy="0 1.57 0" />
       <geometry>
-        <mesh filename="package://ragnar_support/meshes/ragnar_single_arm2.stl" />
+        <cylinder length="0.1" radius="0.04"/>
       </geometry>
       <material name="">
-        <color rgba="0.75 0.75 0.75 1" />
+        <color rgba="0.5 0.5 0.5 1" />
+      </material>
+    </visual>
+    <visual>
+      <origin xyz="0 ${d1/2} 0" rpy="1.57 0 0" />
+      <geometry>
+        <cylinder length="${d1}" radius="0.02"/>
+      </geometry>
+      <material name="">
+        <color rgba="0.5 0.5 0.5 1" />
       </material>
     </visual>
