Commit message: Added complex geometry to urdf and state publisher

File: ragnar_support/urdf/ragnar_macro.xacro (robot description, xacro)
@@ -1,5 +1,5 @@
 <?xml version="1.0" ?>
 <robot name="Ragnar" xmlns:xacro="http://ros.org/wiki/xacro">
-  <xacro:include filename="$(find ragnar_support)/urdf/ragnar_upper2_macro.xacro"/>
+  <xacro:include filename="$(find ragnar_support)/urdf/ragnar_upper3_macro.xacro"/>
   <xacro:macro name="ragnar" params="prefix">
     <!-- Base Link -->
@@ -59,5 +59,5 @@
     <joint name="${prefix}ee_joint" type="floating">
       <origin xyz="0 0 0" rpy="0 0 0" />
-      <parent link="${prefix}lower_arm_1" />
+      <parent link="${prefix}base_link" />
       <child link="${prefix}ee_link" />
     </joint>

Commit message: Lower arms replaced with CAD geometry file

File: ragnar_support/urdf/ragnar_macro.xacro (robot description, xacro)
@@ -42,5 +42,5 @@
     <link name="${prefix}ee_link">
       <visual>
-        <origin xyz="0 0 0" rpy="1.57 0 1.57" />
+        <origin xyz="0 0.019 0" rpy="1.57 0 1.57" />
         <geometry>
           <mesh filename="package://ragnar_support/meshes/ragnar_ee.STL" />

File: ragnar_support/urdf/ragnar_upper3_macro.xacro (robot description, xacro)
@@ -51,5 +51,5 @@
   <link name="${prefix}lower_arm_${num}a">
     <visual>
-      <origin xyz="0 0 0" rpy="0 0 1.57" />
+      <origin xyz="0 0 0" rpy="-1.57 0 1.57" />
       <geometry>
         <mesh filename="package://ragnar_support/meshes/ragnar_single_arm2.stl" />
@@ -76,19 +76,10 @@
   <link name="${prefix}lower_arm_${num}b">
     <visual>
-      <origin xyz="0 0 0" rpy="0 1.57 0" />
+      <origin xyz="0 0 0" rpy="1.57 0 1.57" />
       <geometry>
-        <cylinder length="0.1" radius="0.04"/>
+        <mesh filename="package://ragnar_support/meshes/ragnar_single_arm2.stl" />
       </geometry>
       <material name="">
-        <color rgba="0.5 0.5 0.5 1" />
-      </material>
-    </visual>
-    <visual>
-      <origin xyz="0 ${d1/2} 0" rpy="1.57 0 0" />
-      <geometry>
-        <cylinder length="${d1}" radius="0.02"/>
-      </geometry>
-      <material name="">
-        <color rgba="0.5 0.5 0.5 1" />
+        <color rgba="0.75 0.75 0.75 1" />
       </material>
     </visual>

Commit message: Finished xacro changes for CAD based visualization

File: ragnar_support/urdf/ragnar_macro.xacro (robot description, xacro)
@@ -1,17 +1,10 @@
 <?xml version="1.0" ?>
 <robot name="Ragnar" xmlns:xacro="http://ros.org/wiki/xacro">
-  <xacro:include filename="$(find ragnar_support)/urdf/ragnar_upper3_macro.xacro"/>
+  <xacro:include filename="$(find ragnar_support)/urdf/ragnar_leg_macro.xacro"/>
   <xacro:macro name="ragnar" params="prefix">
     <!-- Base Link -->
-    <link name="${prefix}base_link"/>
-    <link name="${prefix}base_link2">
-      <inertial>
-        <origin xyz="-4.80572213006859E-06 9.64495107789746E-06 -0.0184680705713898" rpy="0 0 0" />
-        <mass value="26.5217124601092" />
-        <inertia ixx="0.936457909215975" ixy="-0.00108838510526368" ixz="1.58187182756307E-06"
-          iyy="1.50216890338436" iyz="1.0107984651762E-05" izz="2.28323593907717" />
-      </inertial>
+    <link name="${prefix}base_link">
       <visual>
-        <origin xyz="0 0 0" rpy="0 0 0" />
+        <origin xyz="0 0 0.045" rpy="0 0 0" />
         <geometry>
           <mesh filename="package://ragnar_support/meshes/base_link.STL" />
@@ -28,15 +21,9 @@
       </collision>
     </link>
-    <joint name="${prefix}base_rotate" type="floating">
-      <origin xyz="0 0 0.05" rpy="0 0 1.5708" />
-      <parent link="${prefix}base_link" />
-      <child link="${prefix}base_link2" />
-      <axis xyz="0 0 0" />
-    </joint>
     <!-- The four ragnar arms -->
-    <xacro:ragnar_upper2 prefix="${prefix}" num="1" x="0.122" y="0.249" z="-0.0877" r="-0.577" p="-0.783" w="-1.311" d1="0.300" d2="0.550"/>
-    <xacro:ragnar_upper2 prefix="${prefix}" num="2" x="-0.122" y="0.249" z="-0.0877" r="-2.698" p="-0.788" w="-1.834" d1="0.300" d2="0.550"/>
-    <xacro:ragnar_upper2 prefix="${prefix}" num="3" x="-0.122" y="-0.249" z="-0.0877" r="-0.456" p="-0.783" w="1.831" d1="0.300" d2="0.550"/>
-    <xacro:ragnar_upper2 prefix="${prefix}" num="4" x="0.122" y="-0.249" z="-0.0877" r="-2.531" p="-0.788" w="1.307" d1="0.300" d2="0.550"/>
+    <xacro:ragnar_leg prefix="${prefix}" num="1" x="0.122" y="0.249" z="-0.0877" r="-0.577" p="-0.783" w="-1.311" d1="0.300" d2="0.550"/>
+    <xacro:ragnar_leg prefix="${prefix}" num="2" x="-0.122" y="0.249" z="-0.0877" r="-2.698" p="-0.788" w="-1.834" d1="0.300" d2="0.550"/>
+    <xacro:ragnar_leg prefix="${prefix}" num="3" x="-0.122" y="-0.249" z="-0.0877" r="-0.456" p="-0.783" w="1.831" d1="0.300" d2="0.550"/>
+    <xacro:ragnar_leg prefix="${prefix}" num="4" x="0.122" y="-0.249" z="-0.0877" r="-2.531" p="-0.788" w="1.307" d1="0.300" d2="0.550"/>
     <!-- End Effector Link -->
     <link name="${prefix}ee_link">
